File: STM32 TEST.kicad_sch (KiCad schematic)
At the start: 33 parts, among them J1 USB_C_Receptacle_USB2.0_16P, J2 SWD, J3 UART 1, J4 I2C 1, J5 SPI 1, J6 Conn_02x10_Odd_Even, J7 Conn_02x10_Odd_Even, SW1 RST, SW2 US 1, U1 STM32F401RETx, U2 AP2112K-3.3, Y1 8MHz

Commit message: Add files via upload
Phase 2
Parts:
- removed J2: SWD, symbol Connector:Conn_01x05_Pin
- removed J5: SPI 1, symbol Connector:Conn_01x06_Pin
- removed U2: AP2112K-3.3, Package_TO_SOT_SMD:SOT-23-5, symbol Regulator_Linear:AP2112K-3.3
- added C1: 2.2uF, Capacitor_SMD:C_0805_2012Metric_Pad1.18x1.45mm_HandSolder, symbol Device:C_Small
- added C13: 4.7uF, Capacitor_SMD:C_0805_2012Metric_Pad1.18x1.45mm_HandSolder, symbol Device:C_Small
- added C14, C16, C19, C20: 100nF, Capacitor_SMD:C_0805_2012Metric_Pad1.18x1.45mm_HandSolder, symbol Device:C_Small
- added C2, C6: 22pF, Capacitor_SMD:C_0805_2012Metric_Pad1.18x1.45mm_HandSolder, symbol Device:C_Small
- added C21: 10uF, Capacitor_SMD:C_0805_2012Metric_Pad1.18x1.45mm_HandSolder, symbol Device:C_Small
- added C5: 8.2pF, Capacitor_SMD:C_0805_2012Metric_Pad1.18x1.45mm_HandSolder, symbol Device:C_Small
- added F1: PTC, Fuse:Fuse_1206_3216Metric_Pad1.42x1.75mm_HandSolder, symbol Device:Polyfuse_Small
- added J3: SWD, Connector_PinHeader_2.54mm:PinHeader_1x06_P2.54mm_Vertical, symbol Connector:Conn_01x06_Pin
- added J6: Micro_SD_Card, Connector_Card:microSD_HC_Hirose_DM3AT-SF-PEJM5, symbol Connector:Micro_SD_Card
- added JP1: SJ1, Jumper:SolderJumper-2_P1.3mm_Bridged_RoundedPad1.0x1.5mm, symbol Jumper:SolderJumper_2_Bridged
- added JP2: SJ2, Jumper:SolderJumper-2_P1.3mm_Bridged_RoundedPad1.0x1.5mm, symbol Jumper:SolderJumper_2_Bridged
- added R10, R11, R9: 10K, Resistor_SMD:R_0805_2012Metric_Pad1.20x1.40mm_HandSolder, symbol Device:R_Small
- added R6, R7: 1K, Resistor_SMD:R_0805_2012Metric_Pad1.20x1.40mm_HandSolder, symbol Device:R_Small
- added SW3: BOOT, Button_Switch_SMD:SW_Push_1TS009xxxx-xxxx-xxxx_6x6x5mm, symbol Switch:SW_Push
- added TP1: 5V, TestPoint:TestPoint_Loop_D2.50mm_Drill1.0mm, symbol Connector:TestPoint
- added TP2: 3V3, TestPoint:TestPoint_Loop_D2.50mm_Drill1.0mm, symbol Connector:TestPoint
- added TP3: GND, TestPoint:TestPoint_Loop_D2.50mm_Drill1.0mm, symbol Connector:TestPoint
- added TP4: VDDA/VREF+, TestPoint:TestPoint_Loop_D2.50mm_Drill1.0mm, symbol Connector:TestPoint
- added TP5: VCAP1, TestPoint:TestPoint_Loop_D2.50mm_Drill1.0mm, symbol Connector:TestPoint
- added TP6: BOOT0, TestPoint:TestPoint_Loop_D2.50mm_Drill1.0mm, symbol Connector:TestPoint
- added TP7: USB D+, TestPoint:TestPoint_Loop_D2.50mm_Drill1.0mm, symbol Connector:TestPoint
- added TP8: USB D-, TestPoint:TestPoint_Loop_D2.50mm_Drill1.0mm, symbol Connector:TestPoint
- added U1: LM66100DCK, Package_TO_SOT_SMD:SOT-363_SC-70-6, symbol Power_Management:LM66100DCK
- added U2: TVS, Package_TO_SOT_SMD:SOT-23-6, symbol Power_Protection:USBLC6-2SC6
- added U4: AP2114H-3.3, Package_TO_SOT_SMD:SOT-223-3_TabPin2, symbol Regulator_Linear:AMS1117-3.3
- added Y1: 8MHz, Crystal:Crystal_SMD_5032-4Pin_5.0x3.2mm, symbol Device:Crystal_GND24
- C10: renamed from C8; footprint (none) -> Capacitor_SMD:C_0805_2012Metric_Pad1.18x1.45mm_HandSolder
- C11: renamed from C7; footprint (none) -> Capacitor_SMD:C_0805_2012Metric_Pad1.18x1.45mm_HandSolder
- C12: renamed from C9; footprint (none) -> Capacitor_SMD:C_0805_2012Metric_Pad1.18x1.45mm_HandSolder
- C15: renamed from C10; footprint (none) -> Capacitor_SMD:C_0805_2012Metric_Pad1.18x1.45mm_HandSolder
- C17: renamed from C5; value 10uF -> 4.7uF; footprint (none) -> Capacitor_SMD:C_0805_2012Metric_Pad1.18x1.45mm_HandSolder
- C18: renamed from C6; footprint (none) -> Capacitor_SMD:C_0805_2012Metric_Pad1.18x1.45mm_HandSolder
- C3: renamed from C11; value 22pF -> 8.2pF; footprint (none) -> Capacitor_SMD:C_0805_2012Metric_Pad1.18x1.45mm_HandSolder
- C4: footprint (none) -> Capacitor_SMD:C_0805_2012Metric_Pad1.18x1.45mm_HandSolder
- C7: renamed from C1; footprint (none) -> Capacitor_SMD:C_0805_2012Metric_Pad1.18x1.45mm_HandSolder
- C8: renamed from C2; footprint (none) -> Capacitor_SMD:C_0805_2012Metric_Pad1.18x1.45mm_HandSolder
- C9: renamed from C3; footprint (none) -> Capacitor_SMD:C_0805_2012Metric_Pad1.18x1.45mm_HandSolder
- D1: renamed from D2; footprint (none) -> LED_SMD:LED_0805_2012Metric_Pad1.15x1.40mm_HandSolder
- D2: renamed from D3; footprint (none) -> LED_SMD:LED_0805_2012Metric_Pad1.15x1.40mm_HandSolder
- D3: renamed from D1; footprint (none) -> LED_SMD:LED_0805_2012Metric_Pad1.15x1.40mm_HandSolder
- FB1: footprint (none) -> Inductor_SMD:L_0805_2012Metric_Pad1.15x1.40mm_HandSolder
- J1: footprint (none) -> Connector_USB:USB_C_Receptacle_HRO_TYPE-C-31-M-12
- J2: renamed from J3; footprint (none) -> Connector_PinHeader_2.54mm:PinHeader_1x04_P2.54mm_Vertical
- J4: footprint (none) -> Connector_PinHeader_2.54mm:PinHeader_1x04_P2.54mm_Vertical
- J5: renamed from J6; value Conn_02x10_Odd_Even -> Conn_Left; footprint (none) -> Connector_PinHeader_2.54mm:PinHeader_2x10_P2.54mm_Vertical
- J7: value Conn_02x10_Odd_Even -> Conn_Right; footprint (none) -> Connector_PinHeader_2.54mm:PinHeader_2x10_P2.54mm_Vertical
- R1: renamed from R2; footprint (none) -> Resistor_SMD:R_0805_2012Metric_Pad1.20x1.40mm_HandSolder
- R2: renamed from R3; footprint (none) -> Resistor_SMD:R_0805_2012Metric_Pad1.20x1.40mm_HandSolder
- R3: renamed from R6; footprint (none) -> Resistor_SMD:R_0805_2012Metric_Pad1.20x1.40mm_HandSolder
- R4, R5: value 22R -> 4.7K; footprint (none) -> Resistor_SMD:R_0805_2012Metric_Pad1.20x1.40mm_HandSolder
- R8: renamed from R1; footprint (none) -> Resistor_SMD:R_0805_2012Metric_Pad1.20x1.40mm_HandSolder
- SW1, SW2: footprint (none) -> Button_Switch_SMD:SW_Push_1TS009xxxx-xxxx-xxxx_6x6x5mm
- Y2: renamed from Y1; value 8MHz -> 32.768 kHz; footprint (none) -> Crystal:Crystal_SMD_3215-2Pin_3.2x1.5mm
- renumbered U1 to U3
Connections:
- net VBAT is gone; now on net +3.3V: U3.1 (VBAT)
- net +3.3V: now also J5.2 (Pin_2), J7.2 (Pin_2), C14.1, C19.1, C20.2, C21.2, J3.1 (Pin_1), J6.4 (VDD), JP1.1 (A), JP2.1 (A), R10.2, R11.2, R9.2, SW3.1, TP2.1, U4.2 (VO); no longer C10.2, C11.2, C12.1, C12.2, C15.1, C17.2, C18.2, C4.2, C7.2, C8.2, C9.2, D1.1 (K), D2.1 (K), D3.1 (K), J1.A1 (GND), J1.A12 (GND), J1.B1 (GND), J1.B12 (GND), J1.S1 (SHIELD), J2.4 (Pin_4), J4.4 (Pin_4), R1.2, R2.2, R3.1, SW1.1, SW1.2, SW2.1, U3.12 (VSSA), U3.18 (VSS), U3.31 (VSS), U3.46 (PA13), U3.47 (VSS), U3.49 (PA14), U3.63 (VSS), U3.7 (NRST)
- net +5V: now also J5.1 (Pin_1), J7.1 (Pin_1), C16.1, TP1.1, U1.6 (VOUT), U2.5 (VBUS), U4.3 (VI); no longer J1.A4 (VBUS), J1.A9 (VBUS), J1.B4 (VBUS), J1.B9 (VBUS)
- net BOOT0: now also SW3.2, TP6.1
- net PA0: now also J5.4 (Pin_4), R7.2
- net PA1: now also J5.5 (Pin_5)
- net PA10: now also J7.6 (Pin_6)
- net PA11: now also U2.6 (I/O1); no longer R4.1
- net PA12: now also U2.4 (I/O2); no longer R5.1
- net PA2: now also J5.6 (Pin_6)
- net PA3: now also J5.7 (Pin_7)
- net PA4: now also J5.8 (Pin_8)
- net PA5: now also J5.9 (Pin_9)
- net PA6: now also J5.10 (Pin_10)
- net PA7: now also J5.11 (Pin_11)
- net PA8: now also J7.4 (Pin_4)
- net PA9: now also J7.5 (Pin_5)
- net PB0: now also J5.18 (Pin_18)
- net PB1: now also J5.19 (Pin_19)
- net PB12: now also J7.13 (Pin_13), J6.2 (DAT3/CD), R11.1
- net PB13: now also J7.14 (Pin_14), J6.5 (CLK)
- net PB14: now also J7.15 (Pin_15), J6.7 (DAT0), R9.1
- net PB15: now also J7.7 (Pin_7), J6.3 (CMD), R10.1
- net PB2: now also J5.20 (Pin_20)
- net PB3: now also J7.8 (Pin_8), J3.6 (Pin_6)
- net PB4: now also J7.9 (Pin_9)
- net PB5: now also J7.10 (Pin_10)
- net PB6: now also J7.11 (Pin_11), R5.2
- net PB7: now also J7.12 (Pin_12), R4.1
- net PC0: now also J5.12 (Pin_12)
- net PC1: now also J5.13 (Pin_13)
- net PC13: now also R6.2; no longer D1.2 (A)
- net PC14: now also C3.1, Y2.2; no longer D2.2 (A)
- net PC15: now also Y2.1, C5.2
- net PC2: now also J5.14 (Pin_14)
- net PC3: now also J5.15 (Pin_15)
- net PC4: now also J5.16 (Pin_16)
- net PC5: now also J5.17 (Pin_17)
- net PC6: now also J7.17 (Pin_17)
- net PC7: now also J7.18 (Pin_18)
- net PC8: now also J7.19 (Pin_19)
- net PC9: now also J7.20 (Pin_20)
- net PH0: now also C2.1, Y1.1; no longer C3.1, Y2.2
- net PH1: now also C6.1, Y1.3; no longer C3.2, Y2.1
- net VCAP1: now also C13.1, TP5.1
- net VREF+: now also TP4.1
- net D-: now reaches J1.A7 (D-), J1.B7 (D-)
- net D-: now also TP8.1, U2.1 (I/O1); no longer R4.2
- net GND: now reaches J7.16 (Pin_16)
- net GND: now also C10.2, C11.2, C12.1, C15.1, C17.2, C18.2, C3.2, C4.2, C7.2, C8.2, C9.2, D1.1 (K), D2.1 (K), D3.1 (K), J1.A1 (GND), J1.A12 (GND), J1.B1 (GND), J1.B12 (GND), J1.S1 (SHIELD), J2.4 (Pin_4), J4.4 (Pin_4), J5.3 (Pin_3), J7.3 (Pin_3), R1.2, R2.2, R3.1, SW1.1, SW2.1, U3.12 (VSSA), U3.18 (VSS), U3.31 (VSS), U3.47 (VSS), U3.63 (VSS), C1.2, C13.2, C14.2, C16.2, C19.2, C2.2, C20.1, C21.1, C5.1, C6.2, J3.3 (Pin_3), J6.6 (VSS), J6.9 (SHIELD), TP3.1, U1.2 (GND), U1.3 (~{CE}), U2.2 (GND), U4.1 (GND), Y1.2, Y1.4
- net D+: now reaches J1.A6 (D+), J1.B6 (D+)
- net D+: now also TP7.1, U2.3 (I/O2); no longer R5.2
- net PA15: no longer names the net of U3.50 (PA15)
- net PB10: no longer names the net of U3.29 (PB10)
- net PB8: no longer names the net of U3.61 (PB8)
- net PB9: no longer names the net of U3.62 (PB9)
- net PC10: no longer names the net of U3.51 (PC10)
- net PC11: no longer names the net of U3.52 (PC11)
- net PC12: no longer names the net of U3.53 (PC12)
- net PD2: no longer names the net of U3.54 (PD2)
- new net: D2.2 (A), R7.1
- new net: C12.2, J3.5 (Pin_5), SW1.2, U3.7 (NRST)
- new net: D1.2 (A), R6.1
- new net: JP2.2 (B), R5.1
- new net: C1.1, F1.1, U1.1 (VIN)
- new net: F1.2, J1.A4 (VBUS), J1.A9 (VBUS), J1.B4 (VBUS), J1.B9 (VBUS)
- new net: JP1.2 (B), R4.2
- new net PA13: J3.4 (Pin_4), U3.46 (PA13)
- new net PA14: J3.2 (Pin_2), U3.49 (PA14)
- no-connect marks 0 -> 13
Other:
- note added: "3V3"
- note added: "CS"
- note added: "ESD PROTECTION"
- note added: "EXT. OSCILLATOR"
- note added: "GND"
- note added: "LSE / RTC OSCILLATOR"
- note added: "MCU I/O EXPANSION HEADERS"
- note added: "MISO"
- note added: "MOSI"
- note added: "NRST"
- note added: "RX1"
- note added: "SCL1"
- note added: "SDA1"
- note added: "SPI MICRO SD STORAGE"
- note added: "SWCLK"
- note added: "SWDIO"
- note added: "SWO"
- note added: "TEST POINTS"
- note added: "TX1"
- note added: "USB/5V POWER INPUT & PROTECTION"
- note removed: "EXT OSC"
- moved on the sheet: C10, C11, C12, C15, C17, C18, C3, C4, C7, C8, C9, D1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
